File: Edgeberry_SenseAndDrive_Cartridge.kicad_pcb (KiCad board)
At the start: 2 copper layers, 51.8 x 63.2 mm, 49 parts, among them J1 Screw_Terminal_01x08, J2 Grove, J3 Conn_01x02_Pin, Q1 BC847, Q10 FQD17P06TM, Q11 BC847, Q12 FQD17P06TM, Q13 BS170, Q14 BS170, Q2 FQD17P06TM, Q3 BC847, Q4 FQD17P06TM, Q5 BC847, Q6 FQD17P06TM, Q7 BC847, Q8 FQD17P06TM, Q9 BC847

Commit message: Version 1.0 cleanup
Parts:
- R1, R11, R3, R5, R7, R9: value 10k -> 3k3
- R13, R14, R15, R16: value R -> 10k
Other:
- board text added: "EDGEBERRY HARDWARE CARTRIDGE"
- board text added: "Sense'n'Drive, Rev. 1.0, mid 2024"
- board text removed: "EDGEBERRY"
- board text removed: "REV.: 1.0, Mid 2024"
- board text removed: "Sense'n'Drive Cartridge"
